File: asphalt88/asphalt88.kicad_sch (KiCad schematic)
At the start: 262 parts, among them J1 TYPE-C-31-M-12, J2 JST_SH, J3 TC2030, SW1 TS-1187A-B-A-B, SW2 TS-1187A-B-A-B, U1 USBLC6-2SC6, U2 TLV75733PDBV, U3 STM32F446RET6, U4 XC6206P332MR-G, Y1 X322516MLB4SI

Commit message: asphalt88: init southpaw layout
Parts:
- removed OL1: OLED, kbd:OLED, symbol kbd:OLED
- added C79: 100n, Capacitor_SMD:C_0402_1005Metric, symbol Device:C
- added HE68: OH49E-S, Package_TO_SOT_SMD:SOT-23-3, symbol HE60:OH49E-S
- added MX68: 1U, HE60:MX-1U, symbol Mechanical:MountingHole
Connections:
- net +3.3VA: now also C79.1, HE68.1 (VCC)
- net GND: now also C79.2, HE68.3 (GND)
- net HE1: now also HE68.2 (OUT)
Other:
- note added: "22 sensors/mx switches for numpad 88 total"
- moved on the sheet: AM1, AM2, AM3, AM4, AM5, AM6, AM7, AM8, AM9, C1, C10, C11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
